Commit message: Modified URDF file

File: urdf/Mattro_heavy_duty.urdf (robot description, URDF)
Before this commit: robot mattro_rovo_2, 1 links, 0 joints
Links:
- added link control_box_link; visual box size=0.4 0.5 0.26
Joints:
- added joint base_to_box: type fixed, parent mattro_base_link, child control_box_link, origin xyz=0.0 0.0 1.0 rpy=0.0 0.0 3.1416

Commit message: Change urdf

File: urdf/Mattro_heavy_duty.urdf (robot description, URDF)
Before this commit: robot mattro_rovo_2, 2 links, 1 joints
Links:
- added link imu_link; visual mesh filename=package://xsens_mti_driver/urdf/MTi_6xx.stl scale=0.001 0.001 0.001
- link control_box_link: geometry visual box size=0.5 0.4 0.2
Joints:
- added joint imu_to_box: type fixed, parent imu_link, child control_box_link, origin xyz=0.0 0.0 0.0 rpy=0.0 0.0 0.0
- joint base_to_box: child control_box_link -> mattro_base_link; origin xyz=0.0 0.0 1.0 rpy=0.0 0.0 3.1416 -> xyz=0.0 0.0 0.0 rpy=0.0 0.0 0.0; parent mattro_base_link -> control_box_link

Commit message: Fixed urdf file

File: urdf/Mattro_heavy_duty.urdf (robot description, URDF)
Before this commit: robot mattro_rovo_2, 3 links, 2 joints
Links:
- link control_box_link: geometry visual mesh filename=package://bock_controller/urdf/Box_400x500x200.stl scale=0.001 0.001 0.001
- link imu_link: geometry visual mesh filename=package://bock_controller/urdf/MTi_6xx.stl scale=0.001 0.001 0.001
